File: se-k1.kicad_sch (KiCad schematic)
At the start: 25 parts, among them J1 USB_C_Receptacle_USB2.0_14P, U1 ESP32-S3-MINI-1U, U3 W25Q16JVSSIQ, U4 AMS1117-3.3

Commit message: upload
Parts:
- added C5, C6, C7: 100nF, Capacitor_SMD:C_0805_2012Metric, symbol Device:C_Small
- added C8: 100nF, Capacitor_SMD:C_0805_2012Metric, symbol Device:C
- added R5, R6, R7, R8: 10k, Resistor_SMD:R_0402_1005Metric, symbol Device:R
- added S11: TS-1088-AR02016, TS-1088-AR02016:SW_TS-1088-AR02016, symbol TS-1088-AR02016:TS-1088-AR02016
- added TP1: TX, TestPoint:TestPoint_Pad_D1.0mm, symbol Connector:TestPoint
- added TP2: RX, TestPoint:TestPoint_Pad_D1.0mm, symbol Connector:TestPoint
- added TP3: 5V, TestPoint:TestPoint_Pad_D1.0mm, symbol Connector:TestPoint
- added TP4: 3V3, TestPoint:TestPoint_Pad_D1.0mm, symbol Connector:TestPoint
- BT1: footprint SMTU2032-LF:BAT_SMTU2032-LF -> Battery:BatteryHolder_Renata_SMTU2032-LF_1x2032
- C1, C3, C4: footprint (none) -> Capacitor_SMD:C_0805_2012Metric
- J1: footprint (none) -> Connector_USB:USB_C_Receptacle_HRO_TYPE-C-31-M-12
- R1, R2, R3, R4: footprint (none) -> Resistor_SMD:R_0402_1005Metric
- U2: footprint (none) -> SLB9670VQ20FW785XUMA1:QFN50P500X500X90-33N
Connections:
- net +3V3: now also U2.22 (VDD), C5.1, C6.2, C7.2, R5.2, R6.2, R7.1, R8.1, TP4.1
- net +5V: now also TP3.1
- net FLASH_CS: now also U1.28 (IO33)
- net GND: now also S1.1, U2.23 (GND), U2.9 (GND), C5.2, C6.1, C7.1, C8.2, S11.1
- net MISO: now also U1.33 (IO37)
- net MOSI: now also U1.31 (IO35)
- net SCLK: now also U1.32 (IO36)
- net at U2.17 (RST): now also R6.1
- net TPM_PIRQ: now reaches U2.18 (PIRQ)
- net TPM_PIRQ: now also U1.34 (IO38), R5.1
- net TPM_CS: now reaches U2.20 (CS)
- net TPM_CS: now also U1.29 (IO34)
- net at U2.7 (PP): now also R7.2
- net at U1.39 (TXD0): now also TP1.1
- net at U1.40 (RXD0): now also TP2.1
- net at U1.45 (EN): now also C8.1, R8.2, S11.2
- no-connect marks 0 -> 20
Other:
- note added: "MCU"
- note added: "TPM 2.0"
- moved on the sheet: C3, C4, U1, U2

Commit message: finish!
Parts:
- removed R7: 10k, Resistor_SMD:R_0402_1005Metric, symbol Device:R
- removed U2: ~, SLB9670VQ20FW785XUMA1:QFN50P500X500X90-33N, symbol tpm:SLB9670
- added U2: SLM9670AQ20FW1311XTMA1, SLM9670AQ20FW1311XTMA1:QFN50P500X500X90-33N, symbol SLM9670AQ20FW1311XTMA1:SLM9670AQ20FW1311XTMA1
- C1, C3, C4, C5, C6: footprint Capacitor_SMD:C_0805_2012Metric -> Capacitor_SMD:C_0402_1005Metric
- C7: value 100nF -> 10uF; footprint Capacitor_SMD:C_0805_2012Metric -> Capacitor_SMD:C_0402_1005Metric
Connections:
- net +3V3: now also C5.2, R5.1, U2.1 (NCI/VDD), U2.14 (NCI/VDD), U2.22 (VDD), U2.8 (VDD); no longer C5.1, R5.2, R6.2
- net GND: now also C5.1, R6.2, U2.10 (NCI), U2.11 (NCI), U2.12 (NCI), U2.13 (NCI), U2.15 (NCI), U2.16 (NCI/GND), U2.2 (GND), U2.23 (GND), U2.25 (NCI), U2.26 (NCI), U2.27 (NCI), U2.28 (NCI), U2.3 (NCI), U2.31 (NCI), U2.32 (GND), U2.4 (NCI), U2.5 (NCI), U2.9 (GND); no longer C5.2
- net MISO: now also U2.24 (MISO)
- net MOSI: now also U2.21 (MOSI)
- net SCLK: now also U2.19 (SCLK)
- net TPM_CS: now also U2.20 (~{CS})
- net TPM_PIRQ: now also U2.18 (~{PIRQ}); no longer R5.1
- net at R6.1: now also U2.7 (PP)
- new net: R5.2, U2.17 (~{RST})
